Commit message: FIX: xacro default arguments removed
- model is now configurable
- new model with support for split config

Removed xacro defaults:
- inorder
- redefine pi

File: hexapod_description/urdf/hexapod_model.xacro (robot description, xacro)
@@ -2,5 +2,4 @@
 <robot xmlns:xacro="http://ros.org/wiki/xacro" name="Golem">
     <!-- parameters -->
-    <xacro:property name="pi" value="3.1415926535897931"/>
     <xacro:property name="body_length_x" value="0.3556"/>
     <xacro:property name="body_length_y" value="0.165"/>

File: hexapod_description/urdf/phantomX_model.xacro (robot description, xacro)
@@ -1,11 +1,10 @@
 <?xml version="1.0" encoding="UTF-8" ?>
 <robot xmlns:xacro="http://ros.org/wiki/xacro" name="phantomX">
-	<!-- parameters -->
-	<xacro:property name="pi" value="3.1415926535897931" />
-	<xacro:property name="body_length_x" value="0.250" />
-	<xacro:property name="body_length_y" value="0.125" />
-	<xacro:property name="coxa_length" value="0.052" />
-	<xacro:property name="femur_length" value="0.065" />
-	<xacro:property name="tibia_length" value="0.133" />
+    <!-- parameters -->
+    <xacro:property name="body_length_x" value="0.250" />
+    <xacro:property name="body_length_y" value="0.125" />
+    <xacro:property name="coxa_length" value="0.052" />
+    <xacro:property name="femur_length" value="0.065" />
+    <xacro:property name="tibia_length" value="0.133" />
     <gazebo>
         <plugin name="gazebo_ros_control" filename="libgazebo_ros_control.so">
@@ -19,15 +18,15 @@
         <origin xyz="0.0 0.0 0.0" rpy="0.0 0.0 0.0" />
     </joint>
-	<link name="body_link">
-			<visual>
-	  			<origin	xyz="0.0 0.0 0.0" rpy="0.0 0.0 0.0" />
-      			<geometry>
-        			<mesh filename="package://hexapod_description/meshes/phantomX/body.stl" scale="0.001 0.001 0.001"/>
-      			</geometry>
-				<material name="">
-					<color rgba="0.7 0.7 0.7 1" />
-				</material>
-			</visual>
-			<collision>
+    <link name="body_link">
+        <visual>
+            <origin xyz="0.0 0.0 0.0" rpy="0.0 0.0 0.0" />
+            <geometry>
+                <mesh filename="package://hexapod_description/meshes/phantomX/body.stl" scale="0.001 0.001 0.001"/>
+            </geometry>
+            <material name="">
+                <color rgba="0.7 0.7 0.7 1" />
+            </material>
+        </visual>
+        <collision>
             <origin xyz="0.0 0.0 0.0" rpy="0.0 0.0 0.0"/>
             <geometry>
@@ -41,8 +40,5 @@
             <origin xyz="0.0 0.0 0.0" rpy="0.0 0.0 0.0" />
             <mass value="0.00001"/>
-            <inertia
-                ixx="1.0" ixy="0.0"  ixz="0.0"
-                iyy="1.0" iyz="0.0"
-                izz="1.0" />
+            <inertia ixx="1.0" ixy="0.0" ixz="0.0" iyy="1.0" iyz="0.0" izz="1.0" />
         </inertial>
     </link>
@@ -50,133 +46,112 @@
         <material>Gazebo/DarkGrey</material>
     </gazebo>
-	<!-- Head Pan and Tilt properties -->
-	<joint name="head_pan_joint" type="revolute">
-		<parent link="body_link"/>
-		<child link="head_pan_link"/>
-		<axis xyz="0.0 0.0 1.0" />
-		<origin xyz="0.145 0.0 0.080" />
-		<limit lower="-${3.14}" upper="${3.14}" effort="10000" velocity="100" />
-	</joint>
-	<link name="head_pan_link">
-        <inertial>
-            <origin xyz="0.0 0.0 0.0" rpy="0.0 0.0 0.0" />
-            <mass value="0.00001"/>
-            <inertia
-                ixx="1.0" ixy="0.0"  ixz="0.0"
-                iyy="1.0" iyz="0.0"
-                izz="1.0" />
-        </inertial>
-    </link>
-	<joint name="head_tilt_joint" type="revolute">
-		<parent link="head_pan_link"/>
-		<child link="head_tilt_link"/>
-		<axis xyz="0.0 1.0 0.0" />
-		<origin xyz="0.0 0.0 0.020" />
-		<limit lower="-${3.14}" upper="${3.14}" effort="10000" velocity="100" />
-	</joint>
-	<link name="head_tilt_link">
-        <inertial>
-            <origin xyz="0.0 0.0 0.0" rpy="0.0 0.0 0.0" />
-            <mass value="0.00001"/>
-            <inertia
-                ixx="1.0" ixy="0.0"  ixz="0.0"
-                iyy="1.0" iyz="0.0"
-                izz="1.0" />
-        </inertial>
-    </link>
-	<!-- Camera properties -->
-	<joint name="camera_rgb_joint" type="fixed">
-		<parent link="head_tilt_link" />
-		<child link="camera_rgb_optical_frame" />
-		<origin xyz="0.0 0.0 0.0" rpy="${pi/2} ${pi} ${pi/2}" />
-	</joint>
-	<link name="camera_rgb_optical_frame">
-        <inertial>
-            <origin xyz="0.0 0.0 0.0" rpy="0.0 0.0 0.0" />
-            <mass value="0.00001"/>
-            <inertia
-                ixx="1.0" ixy="0.0"  ixz="0.0"
-                iyy="1.0" iyz="0.0"
-                izz="1.0" />
-        </inertial>
-    </link>
-	<joint name="camera_depth_joint" type="fixed">
-		<parent link="head_tilt_link" />
-		<child link="camera_depth_optical_frame" />
-		<origin xyz="0.0 0.0 0.0" rpy="${pi/2} ${pi} ${pi/2}" />
-	</joint>
-	<link name="camera_depth_optical_frame" >
-        <inertial>
-            <origin xyz="0.0 0.0 0.0" rpy="0.0 0.0 0.0" />
-            <mass value="0.00001"/>
-            <inertia
-                ixx="1.0" ixy="0.0"  ixz="0.0"
-                iyy="1.0" iyz="0.0"
-                izz="1.0" />
-        </inertial>
-    </link>
-<joint name="camera_depth_frame" type="fixed">
-	<parent link="head_tilt_link" />
-	<child link="camera_depth_frame_link" />
-	<origin xyz="0.0 0.0 0.0" />
-</joint>
-<link name="camera_depth_frame_link" >
-        <inertial>
-            <origin xyz="0.0 0.0 0.0" rpy="0.0 0.0 0.0" />
-            <mass value="0.00001"/>
-            <inertia
-                ixx="1.0" ixy="0.0"  ixz="0.0"
-                iyy="1.0" iyz="0.0"
-                izz="1.0" />
-        </inertial>
-    </link>
-	<!-- IMU properties -->
-	<joint name="imu_joint" type="fixed">
-		<parent link="base_link" />
-		<child link="imu_link" />
-		<origin xyz="0.0 0.0 0.0" rpy="0.0 0.0 0.0" />
-	</joint>
-	<link name="imu_link">
-        <inertial>
-            <origin xyz="0.0 0.0 0.0" rpy="0.0 0.0 0.0" />
-            <mass value="0.00001"/>
-            <inertia
-                ixx="1.0" ixy="0.0"  ixz="0.0"
-                iyy="1.0" iyz="0.0"
-                izz="1.0" />
-        </inertial>
-    </link>
-	<!-- Joint properties -->
-	<xacro:property name="joint_lower_limit" value="-${3.14}" />
-	<xacro:property name="joint_upper_limit" value="${3.14}" />
-	<xacro:property name="joint_effort" value="6.0" />
-	<xacro:property name="joint_velocity" value="0.524" />
-	<!-- Leg macro -->
-	<xacro:macro name="leg" params="side position x y angle axis">
-		<!-- leg position -->
-		<joint name="leg_center_joint_${side}${position}" type="fixed">
-			<origin xyz="${x} ${y} 0.0" rpy="0.0 0.0 0.0" />
-			<parent link="body_link" />
-			<child link="leg_center_${side}${position}" />
-		</joint>
-		<link name="leg_center_${side}${position}" >
-            <inertial>
-                <origin xyz="0.0 0.0 0.0" rpy="0.0 0.0 0.0" />
-                <mass value="0.00001"/>
-                <inertia
-                    ixx="1.0" ixy="0.0"  ixz="0.0"
-                    iyy="1.0" iyz="0.0"
-                    izz="1.0" />
-            </inertial>
-        </link>
-		<!-- coxa -->
-		<joint name="coxa_joint_${side}${position}" type="revolute">
-			<origin xyz="0.0 0.0 0.0" rpy="0.0 0.0 ${angle}" />
-			<parent link="leg_center_${side}${position}" />
-			<child link="coxa_${side}${position}" />
-			<axis xyz="0.0 0.0 1.0" />
-			<limit lower="${joint_lower_limit}" upper="${joint_upper_limit}" effort="${joint_effort}" velocity="${joint_velocity}" />
-		</joint>
-		<transmission name="coxa_transmission_${side}${position}">
+    <!-- Head Pan and Tilt properties -->
+    <joint name="head_pan_joint" type="revolute">
+        <parent link="body_link"/>
+        <child link="head_pan_link"/>
+        <axis xyz="0.0 0.0 1.0" />
+        <origin xyz="0.145 0.0 0.080" />
+        <limit lower="-${3.14}" upper="${3.14}" effort="10000" velocity="100" />
+    </joint>
+    <link name="head_pan_link">
+        <inertial>
+            <origin xyz="0.0 0.0 0.0" rpy="0.0 0.0 0.0" />
+            <mass value="0.00001"/>
+            <inertia ixx="1.0" ixy="0.0" ixz="0.0" iyy="1.0" iyz="0.0" izz="1.0" />
+        </inertial>
+    </link>
+    <joint name="head_tilt_joint" type="revolute">
+        <parent link="head_pan_link"/>
+        <child link="head_tilt_link"/>
+        <axis xyz="0.0 1.0 0.0" />
+        <origin xyz="0.0 0.0 0.020" />
+        <limit lower="-${3.14}" upper="${3.14}" effort="10000" velocity="100" />
+    </joint>
+    <link name="head_tilt_link">
+        <inertial>
+            <origin xyz="0.0 0.0 0.0" rpy="0.0 0.0 0.0" />
+            <mass value="0.00001"/>
+            <inertia ixx="1.0" ixy="0.0" ixz="0.0" iyy="1.0" iyz="0.0" izz="1.0" />
+        </inertial>
+    </link>
+    <!-- Camera properties -->
+    <joint name="camera_rgb_joint" type="fixed">
+        <parent link="head_tilt_link" />
+        <child link="camera_rgb_optical_frame" />
+        <origin xyz="0.0 0.0 0.0" rpy="${pi/2} ${pi} ${pi/2}" />
+    </joint>
+    <link name="camera_rgb_optical_frame">
+        <inertial>
+            <origin xyz="0.0 0.0 0.0" rpy="0.0 0.0 0.0" />
+            <mass value="0.00001"/>
+            <inertia ixx="1.0" ixy="0.0" ixz="0.0" iyy="1.0" iyz="0.0" izz="1.0" />
+        </inertial>
+    </link>
+    <joint name="camera_depth_joint" type="fixed">
+        <parent link="head_tilt_link" />
+        <child link="camera_depth_optical_frame" />
+        <origin xyz="0.0 0.0 0.0" rpy="${pi/2} ${pi} ${pi/2}" />
+    </joint>
+    <link name="camera_depth_optical_frame">
+        <inertial>
+            <origin xyz="0.0 0.0 0.0" rpy="0.0 0.0 0.0" />
+            <mass value="0.00001"/>
+            <inertia ixx="1.0" ixy="0.0" ixz="0.0" iyy="1.0" iyz="0.0" izz="1.0" />
+        </inertial>
+    </link>
+    <joint name="camera_depth_frame" type="fixed">
+        <parent link="head_tilt_link" />
+        <child link="camera_depth_frame_link" />
+        <origin xyz="0.0 0.0 0.0" />
+    </joint>
+    <link name="camera_depth_frame_link">
+        <inertial>
+            <origin xyz="0.0 0.0 0.0" rpy="0.0 0.0 0.0" />
+            <mass value="0.00001"/>
+            <inertia ixx="1.0" ixy="0.0" ixz="0.0" iyy="1.0" iyz="0.0" izz="1.0" />
+        </inertial>
+    </link>
+    <!-- IMU properties -->
+    <joint name="imu_joint" type="fixed">
+        <parent link="base_link" />
+        <child link="imu_link" />
+        <origin xyz="0.0 0.0 0.0" rpy="0.0 0.0 0.0" />
+    </joint>
+    <link name="imu_link">
+        <inertial>
+            <origin xyz="0.0 0.0 0.0" rpy="0.0 0.0 0.0" />
+            <mass value="0.00001"/>
+            <inertia ixx="1.0" ixy="0.0" ixz="0.0" iyy="1.0" iyz="0.0" izz="1.0" />
+        </inertial>
+    </link>
+    <!-- Joint properties -->
+    <xacro:property name="joint_lower_limit" value="-${3.14}" />
+    <xacro:property name="joint_upper_limit" value="${3.14}" />
+    <xacro:property name="joint_effort" value="6.0" />
+    <xacro:property name="joint_velocity" value="0.524" />
+    <!-- Leg macro -->
+    <xacro:macro name="leg" params="side position x y angle axis">
+        <!-- leg position -->
+        <joint name="leg_center_joint_${side}${position}" type="fixed">
+            <origin xyz="${x} ${y} 0.0" rpy="0.0 0.0 0.0" />
+            <parent link="body_link" />
+            <child link="leg_center_${side}${position}" />
+        </joint>
+        <link name="leg_center_${side}${position}">
+            <inertial>
+                <origin xyz="0.0 0.0 0.0" rpy="0.0 0.0 0.0" />
+                <mass value="0.00001"/>
+                <inertia ixx="1.0" ixy="0.0" ixz="0.0" iyy="1.0" iyz="0.0" izz="1.0" />
+            </inertial>
+        </link>
+        <!-- coxa -->
+        <joint name="coxa_joint_${side}${position}" type="revolute">
+            <origin xyz="0.0 0.0 0.0" rpy="0.0 0.0 ${angle}" />
+            <parent link="leg_center_${side}${position}" />
+            <child link="coxa_${side}${position}" />
+            <axis xyz="0.0 0.0 1.0" />
+            <limit lower="${joint_lower_limit}" upper="${joint_upper_limit}" effort="${joint_effort}" velocity="${joint_velocity}" />
+        </joint>
+        <transmission name="coxa_transmission_${side}${position}">
             <type>transmission_interface/SimpleTransmission</type>
             <joint name="coxa_joint_${side}${position}">
@@ -210,8 +185,5 @@
                 <origin xyz="0.0 0.0 0.0" rpy="0.0 0.0 0.0" />
                 <mass value="0.00001"/>
-                <inertia
-                    ixx="1.0" ixy="0.0"  ixz="0.0"
-                    iyy="1.0" iyz="0.0"
-                    izz="1.0" />
+                <inertia ixx="1.0" ixy="0.0" ixz="0.0" iyy="1.0" iyz="0.0" izz="1.0" />
             </inertial>
         </link>
@@ -219,13 +191,13 @@
             <material>Gazebo/DarkGrey</material>
         </gazebo>
-		<!-- femur -->
-		<joint name="femur_joint_${side}${position}" type="revolute">
-			<origin xyz="${coxa_length} 0.0 0.0" rpy="-${pi/2} ${pi/2} 0.0" />
-			<parent link="coxa_${side}${position}" />
-			<child link="femur_${side}${position}" />
-			<axis xyz="0.0 0.0 ${-axis}" />
-			<limit lower="${joint_lower_limit}" upper="${joint_upper_limit}" effort="${joint_effort}" velocity="${joint_velocity}" />
-		</joint>
-		<transmission name="femur_transmission_${side}${position}">
+        <!-- femur -->
+        <joint name="femur_joint_${side}${position}" type="revolute">
+            <origin xyz="${coxa_length} 0.0 0.0" rpy="-${pi/2} ${pi/2} 0.0" />
+            <parent link="coxa_${side}${position}" />
+            <child link="femur_${side}${position}" />
+            <axis xyz="0.0 0.0 ${-axis}" />
+            <limit lower="${joint_lower_limit}" upper="${joint_upper_limit}" effort="${joint_effort}" velocity="${joint_velocity}" />
+        </joint>
+        <transmission name="femur_transmission_${side}${position}">
             <type>transmission_interface/SimpleTransmission</type>
             <joint name="femur_joint_${side}${position}">
@@ -259,8 +231,5 @@
                 <origin xyz="0.0 0.0 0.0" rpy="0.0 0.0 0.0" />
                 <mass value="0.00001"/>
-                <inertia
-                    ixx="1.0" ixy="0.0"  ixz="0.0"
-                    iyy="1.0" iyz="0.0"
-                    izz="1.0" />
+                <inertia ixx="1.0" ixy="0.0" ixz="0.0" iyy="1.0" iyz="0.0" izz="1.0" />
             </inertial>
         </link>
@@ -268,13 +237,13 @@
             <material>Gazebo/DarkGrey</material>
         </gazebo>
-		<!-- tibia -->
-		<joint name="tibia_joint_${side}${position}" type="revolute">
-			<origin xyz="0.0 -${femur_length} 0.0" rpy="${pi} 0.0 0.0" />
-			<parent link="femur_${side}${position}" />
-			<child link="tibia_${side}${position}" />
-			<axis xyz="0.0 0.0 ${axis}" />
-			<limit lower="${joint_lower_limit}" upper="${joint_upper_limit}" effort="${joint_effort}" velocity="${joint_velocity}" />
-		</joint>
-		<transmission name="tibia_transmission_${side}${position}">
+        <!-- tibia -->
+        <joint name="tibia_joint_${side}${position}" type="revolute">
+            <origin xyz="0.0 -${femur_length} 0.0" rpy="${pi} 0.0 0.0" />
+            <parent link="femur_${side}${position}" />
+            <child link="tibia_${side}${position}" />
+            <axis xyz="0.0 0.0 ${axis}" />
+            <limit lower="${joint_lower_limit}" upper="${joint_upper_limit}" effort="${joint_effort}" velocity="${joint_velocity}" />
+        </joint>
+        <transmission name="tibia_transmission_${side}${position}">
             <type>transmission_interface/SimpleTransmission</type>
             <joint name="tibia_joint_${side}${position}">
@@ -308,8 +277,5 @@
                 <origin xyz="0.0 0.0 0.0" rpy="0.0 0.0 0.0" />
                 <mass value="0.00001"/>
-                <inertia
-                    ixx="1.0" ixy="0.0"  ixz="0.0"
-                    iyy="1.0" iyz="0.0"
-                    izz="1.0" />
+                <inertia ixx="1.0" ixy="0.0" ixz="0.0" iyy="1.0" iyz="0.0" izz="1.0" />
             </inertial>
         </link>
@@ -317,11 +283,11 @@
             <material>Gazebo/DarkGrey</material>
         </gazebo>
-	</xacro:macro>
-<!-- Build robot model -->
-	<xacro:leg side="R" position="R" x="-0.120" y="-0.060" angle="-${pi*3/4}" axis="1" />
-	<xacro:leg side="R" position="M" x="0.0" y="-0.100" angle="-${pi/2}" axis="1" />
-	<xacro:leg side="R" position="F" x="0.120" y="-0.060" angle="-${pi/4}" axis="1" />
-	<xacro:leg side="L" position="R" x="-0.120" y="0.060" angle="${pi*3/4}" axis="-1" />
-	<xacro:leg side="L" position="M" x="0.0" y="0.100" angle="${pi/2}" axis="-1" />
-	<xacro:leg side="L" position="F" x="0.120" y="0.060" angle="${pi/4}" axis="-1" />
+    </xacro:macro>
+    <!-- Build robot model -->
+    <xacro:leg side="R" position="R" x="-0.120" y="-0.060" angle="-${pi*3/4}" axis="1" />
+    <xacro:leg side="R" position="M" x="0.0" y="-0.100" angle="-${pi/2}" axis="1" />
+    <xacro:leg side="R" position="F" x="0.120" y="-0.060" angle="-${pi/4}" axis="1" />
+    <xacro:leg side="L" position="R" x="-0.120" y="0.060" angle="${pi*3/4}" axis="-1" />
+    <xacro:leg side="L" position="M" x="0.0" y="0.100" angle="${pi/2}" axis="-1" />
+    <xacro:leg side="L" position="F" x="0.120" y="0.060" angle="${pi/4}" axis="-1" />
 </robot>

File: hexapod_description/urdf/razbot_model.xacro (robot description, xacro)
@@ -3,5 +3,4 @@
 <!--Developed by Shubhankar Das a.k.a Razbotics-->
 	<!-- parameters -->
-	<xacro:property name="pi" value="3.1415926535897931" />
 	<xacro:property name="body_length_x" value="0.294" />
 	<xacro:property name="body_length_y" value="0.340" />
